Commit message: re-built UDRF file. added sample ackermann geometry. added differential drive controller. added ackermann control system (only functional with simplified geometry.

File: description/robot.urdf.xacro (robot description, xacro)
@@ -1,5 +1,7 @@
 <?xml version="1.0" encoding="utf-8"?>
 <robot name="yahboom_bot_1" xmlns:xacro="http://ros.org/wiki/xacro">
-  <xacro:include filename="robot_core.xacro" />
-  <xacro:include filename="gazebo_control.xacro" />
+  <!-- <xacro:include filename="test_ack.xacro" />
+  <xacro:include filename="test_gazebo_ack.xacro" /> -->
+  <xacro:include filename="robot_core_test.xacro" />
+  <xacro:include filename="gazebo_control_diff.xacro" />
 </robot>

File: description/robot_core_test.xacro (robot description, xacro)
@@ -5,7 +5,24 @@
 <robot name="yahboom_bot_1" xmlns:xacro="http://ros.org/wiki/xacro">
   <!--xacro:include filename="$(find yahboomcar_description)/urdf/yahboomcar_R2.gazebo.xacro"/-->
-  <link name="imu_link"/>
+  <!--Colour Descriptions-->
+    <material name="white">
+        <color rgba="1 1 1 1"/>
+    </material>
+    <material name="black">
+        <color rgba="0 0 0 1"/>
+    </material>
+    <material name="grey">
+        <color rgba="0.5 0.5 0.5 1"/>
+    </material>
+  <!--Base Link and Chassis-->
   <link
     name="base_link">
+  </link>
+  <joint name="chassis_joint" type="fixed">
+      <parent link="base_link"/>
+      <child link="chassis"/>
+      <origin xyz="0 0 0"/>
+  </joint>
+  <link name="chassis">
     <inertial>
       <origin
@@ -30,22 +47,17 @@
           filename="package://yahboom_bot_1/meshes/Ackermann/base_link.STL" />
       </geometry>
-      <material
-        name="">
-        <color
-          rgba="0 0.62745 0.23529 1" />
-      </material>
-    </visual>
-    <collision>
-      <origin
-        xyz="0 0 0"
-        rpy="0 0 0" />
-      <geometry>
-        <mesh
-          filename="package://yahboom_bot_1/meshes/Ackermann/base_link.STL" />
-      </geometry>
-    </collision>
-  </link>
-  <link
-    name="back_right_link">
+      <material name="white"/>
+    </visual>
+    <collision>
+      <origin
+        xyz="0 0 0.0125"
+        rpy="0 0 0" />
+      <geometry>
+        <box size="0.35 0.05 0.025" />
+      </geometry>
+    </collision>
+  </link>
+  <!--Back Right Wheel-->
+  <link name="back_right_link">
     <inertial>
       <origin
@@ -70,37 +82,30 @@
           filename="package://yahboom_bot_1/meshes/Ackermann/back_right_link.STL" />
       </geometry>
-      <material
-        name="">
-        <color
-          rgba="0.79216 0.81961 0.93333 1" />
-      </material>
-    </visual>
-    <collision>
-      <origin
-        xyz="0 0 0"
-        rpy="0 0 0" />
-      <geometry>
-        <mesh
-          filename="package://yahboom_bot_1/meshes/Ackermann/back_right_link.STL" />
-      </geometry>
-    </collision>
-  </link>
-  <joint
-    name="back_right_joint"
-    type="continuous">
+      <material name="grey"/>
+    </visual>
+    <collision>
+      <origin
+        xyz="0 0 0"
+        rpy="${pi/2} 0 0" />
+      <geometry>
+        <cylinder radius="0.035" length="0.022" />
+      </geometry>
+    </collision>
+  </link>
+  <joint name="back_right_joint" type="continuous">
     <origin
       xyz="-0.11607 -0.08425 0.0125"
       rpy="0 0 0" />
     <parent
-      link="base_link" />
+      link="chassis" />
     <child
       link="back_right_link" />
     <axis
       xyz="0 1 0" />
-    <dynamics
-      damping="0.05" />
-  </joint>
-  <link
-    name="back_left_link">
+    <!-- <dynamics friction="0.8" damping="0.5" />
+    <limit lower="-3.14159" upper="3.14159" effort="200" velocity="-1" /> -->
+  </joint>
+  <!--Back Left Wheel-->
+  <link name="back_left_link">
     <inertial>
       <origin
@@ -120,42 +125,35 @@
       <origin
         xyz="0 0 0"
-        rpy="0 0 0" />
+        rpy="${pi} 0 0" />
       <geometry>
         <mesh
           filename="package://yahboom_bot_1/meshes/Ackermann/back_right_link.STL" />
       </geometry>
-      <material
-        name="">
-        <color
-          rgba="0.792156862745098 0.819607843137255 0.933333333333333 1" />
-      </material>
-    </visual>
-    <collision>
-      <origin
-        xyz="0 0 0"
-        rpy="0 0 0" />
-      <geometry>
-        <mesh
-          filename="package://yahboom_bot_1/meshes/Ackermann/back_right_link.STL" />
-      </geometry>
-    </collision>
-  </link>
-  <joint
-    name="back_left_joint"
-    type="continuous">
+      <material name="grey"/>
+    </visual>
+    <collision>
+      <origin
+        xyz="0 0 0"
+        rpy="${pi/2} 0 0" />
+      <geometry>
+        <cylinder radius="0.035" length="0.022" />
+      </geometry>
+    </collision>
+  </link>
+  <joint name="back_left_joint" type="continuous">
     <origin
       xyz="-0.11607 0.08425 0.0125"
       rpy="0 0 0" />
     <parent
-      link="base_link" />
+      link="chassis" />
     <child
       link="back_left_link" />
     <axis
       xyz="0 1 0" />
-    <dynamics
-      damping="0.05" />
-  </joint>
-  <link
-    name="front_left_steer">
+    <!-- <dynamics friction="0.8" damping="0.5" />
+    <limit lower="-3.14159" upper="3.14159" effort="200" velocity="-1" /> -->
+  </joint>
+  <!--Front Left Steering Joint-->
+  <link name="front_left_steer">
     <inertial>
       <origin
@@ -181,27 +179,21 @@
       </geometry>
       <material
-        name="">
-        <color
-          rgba="0.082353 0.56078 0 1" />
-      </material>
-    </visual>
-    <collision>
-      <origin
-        xyz="0 0 0"
-        rpy="0 0 0" />
-      <geometry>
-        <mesh
-          filename="package://yahboom_bot_1/meshes/Ackermann/front_left_steer.STL" />
-      </geometry>
-    </collision>
-  </link>
-  <joint
-    name="front_left_steer_joint"
-    type="revolute">
+        name="grey" />
+    </visual>
+    <collision>
+      <origin
+        xyz="0 0 0"
+        rpy="0 0 0" />
+      <geometry>
+        <box size="0.015 0.015 0.015" />
+      </geometry>
+    </collision>
+  </link>
+  <joint name="front_left_steer_joint" type="revolute">
     <origin
       xyz="0.11922 0.065 0.0262"
       rpy="0 0 0" />
     <parent
-      link="base_link" />
+      link="chassis" />
     <child
       link="front_left_steer" />
@@ -213,9 +205,7 @@
       effort="10"
       velocity="1" />
-    <dynamics
-      damping="0.05" />
-  </joint>
-  <link
-    name="front_left_wheel">
+  </joint>
+  <!--Front Left Wheel Joint-->
+  <link name="front_left_wheel">
     <inertial>
       <origin
@@ -235,28 +225,21 @@
       <origin
         xyz="0 0 0"
-        rpy="0 0 0" />
+        rpy="${pi} 0 0" />
       <geometry>
         <mesh
           filename="package://yahboom_bot_1/meshes/Ackermann/back_right_link.STL" />
       </geometry>
-      <material
-        name="">
-        <color
-          rgba="0.79216 0.81961 0.93333 1" />
-      </material>
-    </visual>
-    <collision>
-      <origin
-        xyz="0 0 0"
-        rpy="0 0 0" />
-      <geometry>
-        <mesh
-          filename="package://yahboom_bot_1/meshes/Ackermann/back_right_link.STL" />
-      </geometry>
-    </collision>
-  </link>
-  <joint
-    name="front_left_wheel_joint"
-    type="continuous">
+      <material name="grey"/>
+    </visual>
+    <collision>
+      <origin
+        xyz="0 0 0"
+        rpy="${pi/2} 0 0" />
+      <geometry>
+        <cylinder radius="0.035" length="0.022" />
+      </geometry>
+    </collision>
+  </link>
+  <joint name="front_left_wheel_joint" type="continuous">
     <origin
       xyz="0.00022897 0.0228 -0.0141"
@@ -267,10 +250,10 @@
       link="front_left_wheel" />
     <axis
-      xyz="0 -1 0" />
-    <dynamics
-      damping="0.05" />
-  </joint>
-  <link
-    name="front_right_steer">
+      xyz="0 1 0" />
+    <!-- <dynamics friction="0.8" damping="0.5" />
+    <limit lower="-3.14159" upper="3.14159" effort="200" velocity="-1" /> -->
+  </joint>
+  <!--Front Right Steering Joint-->
+  <link name="front_right_steer">
     <inertial>
       <origin
@@ -290,33 +273,26 @@
       <origin
         xyz="0 0 0"
-        rpy="0 0 0" />
+        rpy="0 0 ${pi}" />
       <geometry>
         <mesh
           filename="package://yahboom_bot_1/meshes/Ackermann/front_left_steer.STL" />
       </geometry>
-      <material
-        name="">
-        <color
-          rgba="0.082353 0.56078 0 1" />
-      </material>
-    </visual>
-    <collision>
-      <origin
-        xyz="0 0 0"
-        rpy="0 0 0" />
-      <geometry>
-        <mesh
-          filename="package://yahboom_bot_1/meshes/Ackermann/front_left_steer.STL" />
-      </geometry>
-    </collision>
-  </link>
-  <joint
-    name="front_right_steer_joint"
-    type="revolute">
+      <material name="grey"/>
+    </visual>
+    <collision>
+      <origin
+        xyz="0 0 0"
+        rpy="0 0 0" />
+      <geometry>
+        <box size="0.015 0.015 0.015" />
+      </geometry>
+    </collision>
+  </link>
+  <joint name="front_right_steer_joint" type="revolute">
     <origin
       xyz="0.11922 -0.065 0.0242"
       rpy="0 0 0" />
     <parent
-      link="base_link" />
+      link="chassis" />
     <child
       link="front_right_steer" />
@@ -328,9 +304,7 @@
       effort="10"
       velocity="1" />
-    <dynamics
-      damping="0.05" />
-  </joint>
-  <link
-    name="front_right_wheel">
+  </joint>
+  <!--Front Right Wheel Joint-->
+  <link name="front_right_wheel">
     <inertial>
       <origin
@@ -355,23 +329,16 @@
           filename="package://yahboom_bot_1/meshes/Ackermann/back_right_link.STL" />
       </geometry>
-      <material
-        name="">
-        <color
-          rgba="0.79216 0.81961 0.93333 1" />
-      </material>
-    </visual>
-    <collision>
-      <origin
-        xyz="0 0 0"
-        rpy="0 0 0" />
-      <geometry>
-        <mesh
-          filename="package://yahboom_bot_1/meshes/Ackermann/back_right_link.STL" />
-      </geometry>
-    </collision>
-  </link>
-  <joint
-    name="front_right_wheel_joint"
-    type="continuous">
+      <material name="grey"/>
+    </visual>
+    <collision>
+      <origin
+        xyz="0 0 0"
+        rpy="${pi/2} 0 0" />
+      <geometry>
+        <cylinder radius="0.035" length="0.022" />
+      </geometry>
+    </collision>
+  </link>
+  <joint name="front_right_wheel_joint" type="continuous">
     <origin
       xyz="-0.00025662 -0.019549 -0.0121"
@@ -383,139 +350,6 @@
     <axis
       xyz="0 1 0" />
-    <dynamics
-      damping="0.05" />
-  </joint>
-  <link
-    name="camera_link">
-    <inertial>
-      <origin
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
File: description/test_gazebo_ack.xacro (robot description, xacro)
@@ -5,25 +5,25 @@
     uses). -->
     <!-- Instead, we need to add gazebo tags for our links that refer to Gazebo materials -->
-    <gazebo reference="chassis">
+    <gazebo reference="chassis_link">
         <material>Gazebo/White</material>
         <mu1>0.5</mu1>
         <mu2>0.5</mu2>
     </gazebo>
-    <gazebo reference="front_left_wheel">
+    <gazebo reference="fr_left_wheel_link">
         <material>Gazebo/Grey</material>
         <mu1>1.0</mu1>
         <mu2>1.0</mu2>
     </gazebo>
-    <gazebo reference="front_right_wheel">
+    <gazebo reference="fr_right_wheel_link">
         <material>Gazebo/Grey</material>
         <mu1>1.0</mu1>
         <mu2>1.0</mu2>
     </gazebo>
-    <gazebo reference="back_left_link">
+    <gazebo reference="re_left_wheel_link">
         <material>Gazebo/Grey</material>
         <mu1>1.0</mu1>
         <mu2>1.0</mu2>
     </gazebo>
-    <gazebo reference="back_right_link">
+    <gazebo reference="re_right_wheel_link">
         <material>Gazebo/Grey</material>
         <mu1>1.0</mu1>
@@ -43,10 +43,10 @@
             filename="libgazebo_ros_joint_state_publisher.so">
             <update_rate>100</update_rate>
-            <joint_name>front_right_steer_joint</joint_name>
-            <joint_name>front_right_wheel_joint</joint_name>
-            <joint_name>front_left_steer_joint</joint_name>
-            <joint_name>front_left_wheel_joint</joint_name>
-            <joint_name>back_right_joint</joint_name>
-            <joint_name>back_left_joint</joint_name>
+            <joint_name>fr_right_steer_joint</joint_name>
+            <joint_name>fr_right_wheel_joint</joint_name>
+            <joint_name>fr_left_steer_joint</joint_name>
+            <joint_name>fr_left_wheel_joint</joint_name>
+            <joint_name>re_right_wheel_joint</joint_name>
+            <joint_name>re_left_wheel_joint</joint_name>
             <joint_name>virtual_steering_wheel_joint</joint_name>
         </plugin>
@@ -74,12 +74,12 @@
                 <remapping>distance:=distance/bot</remapping>
             </ros>
-            <update_rate>100</update_rate>
+            <update_rate>100.0</update_rate>
             <!-- wheels -->
-            <front_left_joint>front_left_wheel_joint</front_left_joint>
-            <front_right_joint>front_right_wheel_joint</front_right_joint>
-            <rear_left_joint>back_left_joint</rear_left_joint>
-            <rear_right_joint>back_right_joint</rear_right_joint>
-            <left_steering_joint>front_left_steer_joint</left_steering_joint>
-            <right_steering_joint>front_right_steer_joint</right_steering_joint>
+            <front_left_joint>fr_left_wheel_joint</front_left_joint>
+            <front_right_joint>fr_right_wheel_joint</front_right_joint>
+            <rear_left_joint>re_left_wheel_joint</rear_left_joint>
+            <rear_right_joint>re_right_wheel_joint</rear_right_joint>
+            <left_steering_joint>fr_left_steer_joint</left_steering_joint>
+            <right_steering_joint>fr_right_steer_joint</right_steering_joint>
             <steering_wheel_joint>virtual_steering_wheel_joint</steering_wheel_joint>
             <!-- Max absolute steer angle for tyre in radians-->
@@ -101,9 +101,9 @@
             <publish_odom_tf>true</publish_odom_tf>     <!-- Don't pubslish this when using robot
             localization -->
-            <publish_wheel_tf>true</publish_wheel_tf>  <!-- Don't publish this. It will override all
+            <publish_wheel_tf>false</publish_wheel_tf>  <!-- Don't publish this. It will override all
             wheel frames to robot_base_frame parameter below.-->
             <publish_distance>true</publish_distance>
             <odometry_frame>odom</odometry_frame>
-            <robot_base_frame>chassis</robot_base_frame>
+            <robot_base_frame>base_footprint</robot_base_frame>
         </plugin>
     </gazebo>
@@ -122,10 +122,10 @@
             <origin xyz="0.0 0.0 0.0" rpy="0.0 0.0 0.0" />
             <mass value="0.001" />
-            <inertia ixx="0.0001" ixy="0.0001" ixz="0.0001" iyy="0.0001" iyz="0.0001" izz="0.0001" />
+            <inertia ixx="0.0" ixy="0.0" ixz="0.0" iyy="0.0" iyz="0.0" izz="0.0" />
         </inertial>
     </link>
     <joint name="virtual_steering_wheel_joint" type="revolute">
         <origin xyz="-0.32 0.0 0.0" rpy="0.0 0.0 0.0" />
-        <parent link="chassis" />
+        <parent link="chassis_link" />
         <child link="virtual_steer_link" />
         <axis xyz="-1 0 0" />
