Commit message: renamed xacro files

File: description/OLD_gazebo_control.xacro (robot description, xacro)
@@ -5,25 +5,25 @@
     uses). -->
     <!-- Instead, we need to add gazebo tags for our links that refer to Gazebo materials -->
-    <gazebo reference="chassis_link">
+    <gazebo reference="chassis">
         <material>Gazebo/White</material>
         <mu1>0.5</mu1>
         <mu2>0.5</mu2>
     </gazebo>
-    <gazebo reference="fr_left_wheel_link">
+    <gazebo reference="front_left_wheel">
         <material>Gazebo/Grey</material>
         <mu1>1.0</mu1>
         <mu2>1.0</mu2>
     </gazebo>
-    <gazebo reference="fr_right_wheel_link">
+    <gazebo reference="front_right_wheel">
         <material>Gazebo/Grey</material>
         <mu1>1.0</mu1>
         <mu2>1.0</mu2>
     </gazebo>
-    <gazebo reference="re_left_wheel_link">
+    <gazebo reference="back_left_link">
         <material>Gazebo/Grey</material>
         <mu1>1.0</mu1>
         <mu2>1.0</mu2>
     </gazebo>
-    <gazebo reference="re_right_wheel_link">
+    <gazebo reference="back_right_link">
         <material>Gazebo/Grey</material>
         <mu1>1.0</mu1>
@@ -43,10 +43,10 @@
             filename="libgazebo_ros_joint_state_publisher.so">
             <update_rate>100</update_rate>
-            <joint_name>fr_right_steer_joint</joint_name>
-            <joint_name>fr_right_wheel_joint</joint_name>
-            <joint_name>fr_left_steer_joint</joint_name>
-            <joint_name>fr_left_wheel_joint</joint_name>
-            <joint_name>re_right_wheel_joint</joint_name>
-            <joint_name>re_left_wheel_joint</joint_name>
+            <joint_name>front_right_steer_joint</joint_name>
+            <joint_name>front_right_wheel_joint</joint_name>
+            <joint_name>front_left_steer_joint</joint_name>
+            <joint_name>front_left_wheel_joint</joint_name>
+            <joint_name>back_right_joint</joint_name>
+            <joint_name>back_left_joint</joint_name>
             <joint_name>virtual_steering_wheel_joint</joint_name>
         </plugin>
@@ -69,26 +69,20 @@
         <plugin name='gazebo_ackermann_drive' filename='libgazebo_ros_ackermann_drive.so'>
             <ros>
-                <!-- <namespace>ugv_gazebo_ackermann</namespace> -->
+                <!-- <namespace>ns_1</namespace> -->
                 <remapping>cmd_vel:=cmd_vel</remapping>
                 <remapping>odom:=odom/bot</remapping>
                 <remapping>distance:=distance/bot</remapping>
             </ros>
-            <update_rate>100.0</update_rate>
-            <!-- wheels -->
-            <front_left_joint>fr_left_wheel_joint</front_left_joint>
-            <front_right_joint>fr_right_wheel_joint</front_right_joint>
-            <rear_left_joint>re_left_wheel_joint</rear_left_joint>
-            <rear_right_joint>re_right_wheel_joint</rear_right_joint>
-            <left_steering_joint>fr_left_steer_joint</left_steering_joint>
-            <right_steering_joint>fr_right_steer_joint</right_steering_joint>
+            <update_rate>100</update_rate>
+            <front_left_joint>front_left_wheel_joint</front_left_joint>
+            <front_right_joint>front_right_wheel_joint</front_right_joint>
+            <rear_left_joint>back_left_joint</rear_left_joint>
+            <rear_right_joint>back_right_joint</rear_right_joint>
+            <left_steering_joint>front_left_steer_joint</left_steering_joint>
+            <right_steering_joint>front_right_steer_joint</right_steering_joint>
             <steering_wheel_joint>virtual_steering_wheel_joint</steering_wheel_joint>
-            <!-- Max absolute steer angle for tyre in radians-->
-            <!-- Any cmd_vel angular z greater than this would be capped -->
             <max_steer>0.383972</max_steer>
-            <!-- Max absolute steering angle of steering wheel -->
             <max_steering_angle>1.570796</max_steering_angle>
-            <!-- Max absolute linear speed in m/s -->
             <max_speed>5</max_speed>
-            <!-- PID tuning -->
             <left_steering_pid_gain>1500 0 1</left_steering_pid_gain>
             <left_steering_i_range>0 0</left_steering_i_range>
@@ -97,13 +91,10 @@
             <linear_velocity_pid_gain>1500 0 1</linear_velocity_pid_gain>
             <linear_velocity_i_range>0 0</linear_velocity_i_range>
-            <!-- output -->
             <publish_odom>true</publish_odom>
-            <publish_odom_tf>true</publish_odom_tf>     <!-- Don't pubslish this when using robot
-            localization -->
-            <publish_wheel_tf>false</publish_wheel_tf>  <!-- Don't publish this. It will override all
-            wheel frames to robot_base_frame parameter below.-->
+            <publish_odom_tf>true</publish_odom_tf>
+            <publish_wheel_tf>false</publish_wheel_tf>
             <publish_distance>true</publish_distance>
-            <odometry_frame>odom</odometry_frame>
-            <robot_base_frame>base_footprint</robot_base_frame>
+            <odometry_frame>chassis</odometry_frame>
+            <robot_base_frame>chassis</robot_base_frame>
         </plugin>
     </gazebo>
@@ -119,5 +110,5 @@
             </material>
         </visual>
-        <inertial>  <!-- Gazebo won't show this link without this inertial mass -->
+        <inertial>
             <origin xyz="0.0 0.0 0.0" rpy="0.0 0.0 0.0" />
             <mass value="0.001" />
@@ -127,5 +118,5 @@
     <joint name="virtual_steering_wheel_joint" type="revolute">
         <origin xyz="-0.32 0.0 0.0" rpy="0.0 0.0 0.0" />
-        <parent link="chassis_link" />
+        <parent link="chassis" />
         <child link="virtual_steer_link" />
         <axis xyz="-1 0 0" />

File: description/gazebo_control.xacro (robot description, xacro)
@@ -5,25 +5,25 @@
     uses). -->
     <!-- Instead, we need to add gazebo tags for our links that refer to Gazebo materials -->
-    <gazebo reference="chassis">
+    <gazebo reference="chassis_link">
         <material>Gazebo/White</material>
         <mu1>0.5</mu1>
         <mu2>0.5</mu2>
     </gazebo>
-    <gazebo reference="front_left_wheel">
+    <gazebo reference="fr_left_wheel_link">
         <material>Gazebo/Grey</material>
         <mu1>1.0</mu1>
         <mu2>1.0</mu2>
     </gazebo>
-    <gazebo reference="front_right_wheel">
+    <gazebo reference="fr_right_wheel_link">
         <material>Gazebo/Grey</material>
         <mu1>1.0</mu1>
         <mu2>1.0</mu2>
     </gazebo>
-    <gazebo reference="back_left_link">
+    <gazebo reference="re_left_wheel_link">
         <material>Gazebo/Grey</material>
         <mu1>1.0</mu1>
         <mu2>1.0</mu2>
     </gazebo>
-    <gazebo reference="back_right_link">
+    <gazebo reference="re_right_wheel_link">
         <material>Gazebo/Grey</material>
         <mu1>1.0</mu1>
@@ -43,10 +43,10 @@
             filename="libgazebo_ros_joint_state_publisher.so">
             <update_rate>100</update_rate>
-            <joint_name>front_right_steer_joint</joint_name>
-            <joint_name>front_right_wheel_joint</joint_name>
-            <joint_name>front_left_steer_joint</joint_name>
-            <joint_name>front_left_wheel_joint</joint_name>
-            <joint_name>back_right_joint</joint_name>
-            <joint_name>back_left_joint</joint_name>
+            <joint_name>fr_right_steer_joint</joint_name>
+            <joint_name>fr_right_wheel_joint</joint_name>
+            <joint_name>fr_left_steer_joint</joint_name>
+            <joint_name>fr_left_wheel_joint</joint_name>
+            <joint_name>re_right_wheel_joint</joint_name>
+            <joint_name>re_left_wheel_joint</joint_name>
             <joint_name>virtual_steering_wheel_joint</joint_name>
         </plugin>
@@ -69,20 +69,26 @@
         <plugin name='gazebo_ackermann_drive' filename='libgazebo_ros_ackermann_drive.so'>
             <ros>
-                <!-- <namespace>ns_1</namespace> -->
+                <!-- <namespace>ugv_gazebo_ackermann</namespace> -->
                 <remapping>cmd_vel:=cmd_vel</remapping>
                 <remapping>odom:=odom/bot</remapping>
                 <remapping>distance:=distance/bot</remapping>
             </ros>
-            <update_rate>100</update_rate>
-            <front_left_joint>front_left_wheel_joint</front_left_joint>
-            <front_right_joint>front_right_wheel_joint</front_right_joint>
-            <rear_left_joint>back_left_joint</rear_left_joint>
-            <rear_right_joint>back_right_joint</rear_right_joint>
-            <left_steering_joint>front_left_steer_joint</left_steering_joint>
-            <right_steering_joint>front_right_steer_joint</right_steering_joint>
+            <update_rate>100.0</update_rate>
+            <!-- wheels -->
+            <front_left_joint>fr_left_wheel_joint</front_left_joint>
+            <front_right_joint>fr_right_wheel_joint</front_right_joint>
+            <rear_left_joint>re_left_wheel_joint</rear_left_joint>
+            <rear_right_joint>re_right_wheel_joint</rear_right_joint>
+            <left_steering_joint>fr_left_steer_joint</left_steering_joint>
+            <right_steering_joint>fr_right_steer_joint</right_steering_joint>
             <steering_wheel_joint>virtual_steering_wheel_joint</steering_wheel_joint>
+            <!-- Max absolute steer angle for tyre in radians-->
+            <!-- Any cmd_vel angular z greater than this would be capped -->
             <max_steer>0.383972</max_steer>
+            <!-- Max absolute steering angle of steering wheel -->
             <max_steering_angle>1.570796</max_steering_angle>
+            <!-- Max absolute linear speed in m/s -->
             <max_speed>5</max_speed>
+            <!-- PID tuning -->
             <left_steering_pid_gain>1500 0 1</left_steering_pid_gain>
             <left_steering_i_range>0 0</left_steering_i_range>
@@ -91,10 +97,13 @@
             <linear_velocity_pid_gain>1500 0 1</linear_velocity_pid_gain>
             <linear_velocity_i_range>0 0</linear_velocity_i_range>
+            <!-- output -->
             <publish_odom>true</publish_odom>
-            <publish_odom_tf>true</publish_odom_tf>
-            <publish_wheel_tf>false</publish_wheel_tf>
+            <publish_odom_tf>true</publish_odom_tf>     <!-- Don't pubslish this when using robot
+            localization -->
+            <publish_wheel_tf>false</publish_wheel_tf>  <!-- Don't publish this. It will override all
+            wheel frames to robot_base_frame parameter below.-->
             <publish_distance>true</publish_distance>
-            <odometry_frame>chassis</odometry_frame>
-            <robot_base_frame>chassis</robot_base_frame>
+            <odometry_frame>odom</odometry_frame>
+            <robot_base_frame>base_footprint</robot_base_frame>
         </plugin>
     </gazebo>
@@ -110,5 +119,5 @@
             </material>
         </visual>
-        <inertial>
+        <inertial>  <!-- Gazebo won't show this link without this inertial mass -->
             <origin xyz="0.0 0.0 0.0" rpy="0.0 0.0 0.0" />
             <mass value="0.001" />
@@ -118,5 +127,5 @@
     <joint name="virtual_steering_wheel_joint" type="revolute">
         <origin xyz="-0.32 0.0 0.0" rpy="0.0 0.0 0.0" />
-        <parent link="chassis" />
+        <parent link="chassis_link" />
         <child link="virtual_steer_link" />
         <axis xyz="-1 0 0" />

File: description/robot.urdf.xacro (robot description, xacro)
@@ -1,7 +1,7 @@
 <?xml version="1.0" encoding="utf-8"?>
 <robot name="yahboom_bot_1" xmlns:xacro="http://ros.org/wiki/xacro">
-  <xacro:include filename="TEST_ack_tweak.xacro" />
-  <xacro:include filename="TEST_gazebo_ack.xacro" />
-  <!-- <xacro:include filename="robot_core.xacro" />
-  <xacro:include filename="gazebo_control.xacro" /> -->
+  <!-- <xacro:include filename="TEST_ack_tweak.xacro" />
+  <xacro:include filename="TEST_gazebo_ack.xacro" /> -->
+  <xacro:include filename="robot_core.xacro" />
+  <xacro:include filename="gazebo_control.xacro" />
 </robot>
