Commit message: renamed xacro files

File: description/robot_core.xacro (robot description, xacro)
@@ -1,363 +1,252 @@
-<?xml version="1.0" encoding="utf-8"?>
-<!-- This URDF was automatically created by SolidWorks to URDF Exporter! Originally created by Stephen Brawner (brawner@gmail.com)
-     Commit Version: 1.5.1-0-g916b5db  Build Version: 1.5.7152.31018
-     For more information, please see http://wiki.ros.org/sw_urdf_exporter -->
-<robot name="yahboom_bot_1" xmlns:xacro="http://ros.org/wiki/xacro">
-  <!--xacro:include filename="$(find yahboomcar_description)/urdf/yahboomcar_R2.gazebo.xacro"/-->
-  <!--Colour Descriptions-->
-    <material name="white">
-        <color rgba="1 1 1 1"/>
-    </material>
-    <material name="black">
-        <color rgba="0 0 0 1"/>
-    </material>
-    <material name="grey">
-        <color rgba="0.5 0.5 0.5 1"/>
-    </material>
-  <!--Base Link and Chassis-->
-  <link name="base_footprint">
-    <origin xyz="0 0 0" rpy="0 0 0" />
-  </link>
-  <link name="base_link">
-  </link>
-  <joint name="base_joint" type="fixed">
-      <parent link="base_footprint" />
-      <child link="base_link" />
-      <origin xyz="0.0 0.0 0.0" rpy="0 0 0" />
-  </joint>
-  <joint name="chassis_joint" type="fixed">
-      <parent link="base_link"/>
-      <child link="chassis"/>
-      <origin xyz="0 0 0"/>
-  </joint>
-  <link name="chassis">
-    <inertial>
-      <origin
-        xyz="-0.014025 -0.00011707 0.082168"
-        rpy="0 0 0" />
-      <mass
-        value="0.52447" />
-      <inertia
-        ixx="0.00066245"
-        ixy="-3.1852E-08"
-        ixz="-4.6503E-05"
-        iyy="0.0012486"
-        iyz="-3.356E-08"
-        izz="0.0018052" />
-    </inertial>
-    <visual>
-      <origin
-        xyz="0 0 0"
-        rpy="0 0 0" />
-      <geometry>
-        <mesh
-          filename="package://yahboom_bot_1/meshes/Ackermann/base_link.STL" />
-      </geometry>
-      <material name="white"/>
-    </visual>
-    <collision>
-      <origin
-        xyz="0 0 0.0125"
-        rpy="0 0 0" />
-      <geometry>
-        <box size="0.35 0.05 0.025" />
-      </geometry>
-    </collision>
-  </link>
-  <!--Back Right Wheel-->
-  <link name="back_right_link">
-    <inertial>
-      <origin
-        xyz="3.8959E-08 0.0015615 -6.3774E-08"
-        rpy="0 0 0" />
-      <mass
-        value="0.060236" />
-      <inertia
-        ixx="2.5326E-05"
-        ixy="-2.701E-10"
-        ixz="3.3546E-09"
-        iyy="4.4342E-05"
-        iyz="-2.9324E-10"
-        izz="2.531E-05" />
-    </inertial>
-    <visual>
-      <origin
-        xyz="0 0 0"
-        rpy="0 0 0" />
-      <geometry>
-        <mesh
-          filename="package://yahboom_bot_1/meshes/Ackermann/back_right_link.STL" />
-      </geometry>
-      <material name="grey"/>
-    </visual>
-    <collision>
-      <origin
-        xyz="0 0 0"
-        rpy="${pi/2} 0 0" />
-      <geometry>
-        <cylinder radius="0.035" length="0.022" />
-      </geometry>
-    </collision>
-  </link>
-  <joint name="back_right_joint" type="continuous">
-    <origin
-      xyz="-0.11607 -0.08425 0.0125"
-      rpy="0 0 0" />
-    <parent
-      link="chassis" />
-    <child
-      link="back_right_link" />
-    <axis
-      xyz="0 1 0" />
-    <dynamics friction="0.8" damping="0.5" />
-    <limit lower="-3.14159" upper="3.14159" effort="200" velocity="-1" />
-  </joint>
-  <!--Back Left Wheel-->
-  <link name="back_left_link">
-    <inertial>
-      <origin
-        xyz="-6.87042718550135E-08 -0.00156153690070754 3.00324059371304E-08"
-        rpy="0 0 0" />
-      <mass
-        value="0.0602360431220635" />
-      <inertia
-        ixx="2.53100986719244E-05"
-        ixy="-3.65138701967536E-11"
-        ixz="1.15601374112124E-09"
-        iyy="4.43431918315874E-05"
-        iyz="-7.01985398840287E-11"
-        izz="2.53280330627738E-05" />
-    </inertial>
-    <visual>
-      <origin
-        xyz="0 0 0"
-        rpy="${pi} 0 0" />
-      <geometry>
-        <mesh
-          filename="package://yahboom_bot_1/meshes/Ackermann/back_right_link.STL" />
-      </geometry>
-      <material name="grey"/>
-    </visual>
-    <collision>
-      <origin
-        xyz="0 0 0"
-        rpy="${pi/2} 0 0" />
-      <geometry>
-        <cylinder radius="0.035" length="0.022" />
-      </geometry>
-    </collision>
-  </link>
-  <joint name="back_left_joint" type="continuous">
-    <origin
-      xyz="-0.11607 0.08425 0.0125"
-      rpy="0 0 0" />
-    <parent
-      link="chassis" />
-    <child
-      link="back_left_link" />
-    <axis
-      xyz="0 1 0" />
-    <dynamics friction="0.8" damping="0.5" />
-    <limit lower="-3.14159" upper="3.14159" effort="200" velocity="-1" />
-  </joint>
-  <!--Front Left Steering Joint-->
-  <link name="front_left_steer">
-    <inertial>
-      <origin
-        xyz="-0.0044676 0.0031203 -0.014101"
-        rpy="0 0 0" />
-      <mass
-        value="0.002176" />
-      <inertia
-        ixx="1.4001E-07"
-        ixy="-7.8357E-08"
-        ixz="1.1741E-12"
-        iyy="2.7801E-07"
-        iyz="7.8069E-12"
-        izz="2.909E-07" />
-    </inertial>
-    <visual>
-      <origin
-        xyz="0 0 0"
-        rpy="0 0 0" />
-      <geometry>
-        <mesh
-          filename="package://yahboom_bot_1/meshes/Ackermann/front_left_steer.STL" />
-      </geometry>
-      <material
-        name="grey" />
-    </visual>
-    <collision>
-      <origin
-        xyz="0 0 0"
-        rpy="0 0 0" />
-      <geometry>
-        <mesh
-          filename="package://yahboom_bot_1/meshes/Ackermann/front_left_steer.STL" />
-      </geometry>
-    </collision>
-  </link>
-  <joint name="front_left_steer_joint" type="revolute">
-    <origin
-      xyz="0.11922 0.065 0.0262"
-      rpy="0 0 0" />
-    <parent
-      link="chassis" />
-    <child
-      link="front_left_steer" />
-    <axis
-      xyz="0 0 1" />
-    <limit
-      lower="-0.6"
-      upper="0.6"
-      effort="10"
-      velocity="1" />
-  </joint>
-  <!--Front Left Wheel Joint-->
-  <link name="front_left_wheel">
-    <inertial>
-      <origin
-        xyz="-6.1417E-08 -0.0048115 4.113E-08"
-        rpy="0 0 0" />
-      <mass
-        value="0.060236" />
-      <inertia
-        ixx="2.531E-05"
-        ixy="2.9987E-10"
-        ixz="3.7781E-09"
-        iyy="4.4342E-05"
-        iyz="2.6181E-10"
-        izz="2.5326E-05" />
-    </inertial>
-    <visual>
-      <origin
-        xyz="0 0 0"
-        rpy="${pi} 0 0" />
-      <geometry>
-        <mesh
-          filename="package://yahboom_bot_1/meshes/Ackermann/back_right_link.STL" />
-      </geometry>
-      <material name="grey"/>
-    </visual>
-    <collision>
-      <origin
-        xyz="0 0 0"
-        rpy="${pi/2} 0 0" />
-      <geometry>
-        <cylinder radius="0.035" length="0.022" />
-      </geometry>
-    </collision>
-  </link>
-  <joint name="front_left_wheel_joint" type="continuous">
-    <origin
-      xyz="0.00022897 0.0228 -0.0141"
-      rpy="0 0 -0.010042" />
-    <parent
-      link="front_left_steer" />
-    <child
-      link="front_left_wheel" />
-    <axis
-      xyz="0 1 0" />
-    <dynamics friction="0.8" damping="0.5" />
-    <limit lower="-3.14159" upper="3.14159" effort="200" velocity="-1" />
-  </joint>
-  <!--Front Right Steering Joint-->
-  <link name="front_right_steer">
-    <inertial>
-      <origin
-        xyz="-0.0045387 -0.0030159 -0.012099"
-        rpy="0 0 0" />
-      <mass
-        value="0.002176" />
-      <inertia
-        ixx="1.4372E-07"
-        ixy="8.1469E-08"
-        ixz="-1.0492E-12"
-        iyy="2.7431E-07"
-        iyz="7.8675E-12"
-        izz="2.909E-07" />
-    </inertial>
-    <visual>
-      <origin
-        xyz="0 0 0"
-        rpy="0 0 ${pi}" />
-      <geometry>
-        <mesh
-          filename="package://yahboom_bot_1/meshes/Ackermann/front_left_steer.STL" />
-      </geometry>
-      <material name="grey"/>
-    </visual>
-    <collision>
-      <origin
-        xyz="0 0 0"
-        rpy="0 0 0" />
-      <geometry>
-        <box size="0.015 0.015 0.015" />
-      </geometry>
-    </collision>
-  </link>
-  <joint name="front_right_steer_joint" type="revolute">
-    <origin
-      xyz="0.11922 -0.065 0.0242"
-      rpy="0 0 0" />
-    <parent
-      link="chassis" />
-    <child
-      link="front_right_steer" />
-    <axis
-      xyz="0 0 1" />
-    <limit
-      lower="-0.6"
-      upper="0.6"
-      effort="10"
-      velocity="1" />
-  </joint>
-  <!--Front Right Wheel Joint-->
-  <link name="front_right_wheel">
-    <inertial>
-      <origin
-        xyz="5.5753E-08 0.0015615 -5.0453E-08"
-        rpy="0 0 0" />
-      <mass
-        value="0.060236" />
-      <inertia
-        ixx="2.5325E-05"
-        ixy="5.201E-11"
-        ixz="7.1484E-09"
-        iyy="4.4343E-05"
-        iyz="6.0924E-11"
-        izz="2.5314E-05" />
-    </inertial>
-    <visual>
-      <origin
-        xyz="0 0 0"
-        rpy="0 0 0" />
-      <geometry>
-        <mesh
-          filename="package://yahboom_bot_1/meshes/Ackermann/back_right_link.STL" />
-      </geometry>
-      <material name="grey"/>
-    </visual>
-    <collision>
-      <origin
-        xyz="0 0 0"
-        rpy="${pi/2} 0 0" />
-      <geometry>
-        <cylinder radius="0.035" length="0.022" />
-      </geometry>
-    </collision>
-  </link>
-  <joint name="front_right_wheel_joint" type="continuous">
-    <origin
-      xyz="-0.00025662 -0.019549 -0.0121"
-      rpy="0 0 -0.013126" />
-    <parent
-      link="front_right_steer" />
-    <child
-      link="front_right_wheel" />
-    <axis
-      xyz="0 1 0" />
-    <dynamics friction="0.8" damping="0.5" />
-    <limit lower="-3.14159" upper="3.14159" effort="200" velocity="-1" />
-  </joint>
+<?xml version="1.0"?>
+<robot xmlns:xacro="http://www.ros.org/wiki/xacro">
+    <xacro:property name="body_mass" value="25.0" />
+    <xacro:property name="body_width" value="0.3" />
+    <xacro:property name="body_length" value="0.10" />
+    <xacro:property name="body_depth" value="0.75" />
+    <xacro:property name="wheel_radius" value="0.14" />
+    <xacro:property name="wheel_thickness" value="0.14" />
+    <xacro:property name="wheel_mass" value="3.0" />
+    <xacro:property name="steering_mass" value="0.01" />
+    <!-- BASE -->
+    <link name="base_footprint">
+            <origin xyz="0 0 0" rpy="0 0 0" />
+    </link>
+    <link name="base_link">
+    </link>
+    <joint name="base_joint" type="fixed">
+        <parent link="base_footprint" />
+        <child link="base_link" />
+        <origin xyz="0.0 0.0 0.0" rpy="0 0 0" />
+    </joint>
+    <link name="chassis_link">
+        <inertial>
+            <origin xyz="0 0 0" rpy="0 0 0" />
+            <mass value="24.73" />
+            <inertia ixx="${body_mass/12 * (body_width*body_width + body_length*body_length)}"
+                ixy="0" ixz="0"
+                iyy="${body_mass/12 * (body_length*body_length + body_depth*body_depth)}" iyz="0"
+                izz="${body_mass/12 * (body_width*body_width + body_depth*body_depth)}" />
+        </inertial>
+        <visual>
+            <origin xyz="0 0 0" rpy="0 0 0" />
+            <geometry>
+                <mesh
+                filename="package://yahboom_bot_1/meshes/Ackermann/base_link.STL" />
+            </geometry>
+        </visual>
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