Commit message: Ackermann steering control system successfully linked with Yahboom Geometry!

File: description/gazebo_control.xacro (robot description, xacro)
@@ -69,5 +69,5 @@
         <plugin name='gazebo_ackermann_drive' filename='libgazebo_ros_ackermann_drive.so'>
             <ros>
-                <!-- <namespace>ugv_gazebo_ackermann</namespace> -->
+                <!-- <namespace>ns_1</namespace> -->
                 <remapping>cmd_vel:=cmd_vel</remapping>
                 <remapping>odom:=odom/bot</remapping>
@@ -75,5 +75,4 @@
             </ros>
             <update_rate>100</update_rate>
-            <!-- wheels -->
             <front_left_joint>front_left_wheel_joint</front_left_joint>
             <front_right_joint>front_right_wheel_joint</front_right_joint>
@@ -83,12 +82,7 @@
             <right_steering_joint>front_right_steer_joint</right_steering_joint>
             <steering_wheel_joint>virtual_steering_wheel_joint</steering_wheel_joint>
-            <!-- Max absolute steer angle for tyre in radians-->
-            <!-- Any cmd_vel angular z greater than this would be capped -->
             <max_steer>0.383972</max_steer>
-            <!-- Max absolute steering angle of steering wheel -->
             <max_steering_angle>1.570796</max_steering_angle>
-            <!-- Max absolute linear speed in m/s -->
             <max_speed>5</max_speed>
-            <!-- PID tuning -->
             <left_steering_pid_gain>1500 0 1</left_steering_pid_gain>
             <left_steering_i_range>0 0</left_steering_i_range>
@@ -97,12 +91,9 @@
             <linear_velocity_pid_gain>1500 0 1</linear_velocity_pid_gain>
             <linear_velocity_i_range>0 0</linear_velocity_i_range>
-            <!-- output -->
             <publish_odom>true</publish_odom>
-            <publish_odom_tf>true</publish_odom_tf>     <!-- Don't pubslish this when using robot
-            localization -->
-            <publish_wheel_tf>true</publish_wheel_tf>  <!-- Don't publish this. It will override all
-            wheel frames to robot_base_frame parameter below.-->
+            <publish_odom_tf>true</publish_odom_tf>
+            <publish_wheel_tf>false</publish_wheel_tf>
             <publish_distance>true</publish_distance>
-            <odometry_frame>odom</odometry_frame>
+            <odometry_frame>chassis</odometry_frame>
             <robot_base_frame>chassis</robot_base_frame>
         </plugin>
@@ -119,8 +110,8 @@
             </material>
         </visual>
-        <inertial>  <!-- Gazebo won't show this link without this inertial mass -->
+        <inertial>
             <origin xyz="0.0 0.0 0.0" rpy="0.0 0.0 0.0" />
             <mass value="0.001" />
-            <inertia ixx="0.0001" ixy="0.0001" ixz="0.0001" iyy="0.0001" iyz="0.0001" izz="0.0001" />
+            <inertia ixx="0.0" ixy="0.0" ixz="0.0" iyy="0.0" iyz="0.0" izz="0.0" />
         </inertial>
     </link>

File: description/gazebo_control_diff.xacro (robot description, xacro)
@@ -1,4 +1,23 @@
 <?xml version="1.0"?>
 <robot xmlns:xacro="http://www.ros.org/wiki/xacro">
+    <gazebo>
+        <plugin name="gazebo_ros_joint_state_publisher"
+            filename="libgazebo_ros_joint_state_publisher.so">
+            <update_rate>100</update_rate>
+            <joint_name>front_right_steer_joint</joint_name>
+            <joint_name>front_right_wheel_joint</joint_name>
+            <joint_name>front_left_steer_joint</joint_name>
+            <joint_name>front_left_wheel_joint</joint_name>
+            <joint_name>back_right_joint</joint_name>
+            <joint_name>back_left_joint</joint_name>
+            <joint_name>virtual_steering_wheel_joint</joint_name>
+        </plugin>
+    </gazebo>
+    <gazebo>
+        <plugin name="gazebo_ros_joint_pose_trajectory"
+            filename="libgazebo_ros_joint_pose_trajectory.so">
+            <update_rate>2</update_rate>
+        </plugin>
+    </gazebo>
    <gazebo>
         <plugin name="diff_drive" filename="libgazebo_ros_diff_drive.so">

File: description/robot.urdf.xacro (robot description, xacro)
@@ -1,7 +1,7 @@
 <?xml version="1.0" encoding="utf-8"?>
 <robot name="yahboom_bot_1" xmlns:xacro="http://ros.org/wiki/xacro">
-  <!-- <xacro:include filename="test_ack.xacro" />
-  <xacro:include filename="test_gazebo_ack.xacro" /> -->
-  <xacro:include filename="robot_core_test.xacro" />
-  <xacro:include filename="gazebo_control_diff.xacro" />
+  <xacro:include filename="TEST_ack_tweak.xacro" />
+  <xacro:include filename="TEST_gazebo_ack.xacro" />
+  <!-- <xacro:include filename="robot_core.xacro" />
+  <xacro:include filename="gazebo_control.xacro" /> -->
 </robot>

File: description/robot_core.xacro (robot description, xacro)
@@ -5,7 +5,31 @@
 <robot name="yahboom_bot_1" xmlns:xacro="http://ros.org/wiki/xacro">
   <!--xacro:include filename="$(find yahboomcar_description)/urdf/yahboomcar_R2.gazebo.xacro"/-->
-  <link name="imu_link"/>
-  <link
-    name="base_link">
+  <!--Colour Descriptions-->
+    <material name="white">
+        <color rgba="1 1 1 1"/>
+    </material>
+    <material name="black">
+        <color rgba="0 0 0 1"/>
+    </material>
+    <material name="grey">
+        <color rgba="0.5 0.5 0.5 1"/>
+    </material>
+  <!--Base Link and Chassis-->
+  <link name="base_footprint">
+    <origin xyz="0 0 0" rpy="0 0 0" />
+  </link>
+  <link name="base_link">
+  </link>
+  <joint name="base_joint" type="fixed">
+      <parent link="base_footprint" />
+      <child link="base_link" />
+      <origin xyz="0.0 0.0 0.0" rpy="0 0 0" />
+  </joint>
+  <joint name="chassis_joint" type="fixed">
+      <parent link="base_link"/>
+      <child link="chassis"/>
+      <origin xyz="0 0 0"/>
+  </joint>
+  <link name="chassis">
     <inertial>
       <origin
@@ -30,22 +54,17 @@
           filename="package://yahboom_bot_1/meshes/Ackermann/base_link.STL" />
       </geometry>
-      <material
-        name="">
-        <color
-          rgba="0 0.62745 0.23529 1" />
-      </material>
-    </visual>
-    <collision>
-      <origin
-        xyz="0 0 0"
-        rpy="0 0 0" />
-      <geometry>
-        <mesh
-          filename="package://yahboom_bot_1/meshes/Ackermann/base_link.STL" />
-      </geometry>
-    </collision>
-  </link>
-  <link
-    name="back_right_link">
+      <material name="white"/>
+    </visual>
+    <collision>
+      <origin
+        xyz="0 0 0.0125"
+        rpy="0 0 0" />
+      <geometry>
+        <box size="0.35 0.05 0.025" />
+      </geometry>
+    </collision>
+  </link>
+  <!--Back Right Wheel-->
+  <link name="back_right_link">
     <inertial>
       <origin
@@ -70,37 +89,30 @@
           filename="package://yahboom_bot_1/meshes/Ackermann/back_right_link.STL" />
       </geometry>
-      <material
-        name="">
-        <color
-          rgba="0.79216 0.81961 0.93333 1" />
-      </material>
-    </visual>
-    <collision>
-      <origin
-        xyz="0 0 0"
-        rpy="0 0 0" />
-      <geometry>
-        <mesh
-          filename="package://yahboom_bot_1/meshes/Ackermann/back_right_link.STL" />
-      </geometry>
-    </collision>
-  </link>
-  <joint
-    name="back_right_joint"
-    type="continuous">
+      <material name="grey"/>
+    </visual>
+    <collision>
+      <origin
+        xyz="0 0 0"
+        rpy="${pi/2} 0 0" />
+      <geometry>
+        <cylinder radius="0.035" length="0.022" />
+      </geometry>
+    </collision>
+  </link>
+  <joint name="back_right_joint" type="continuous">
     <origin
       xyz="-0.11607 -0.08425 0.0125"
       rpy="0 0 0" />
     <parent
-      link="base_link" />
+      link="chassis" />
     <child
       link="back_right_link" />
     <axis
       xyz="0 1 0" />
-    <dynamics
-      damping="0.05" />
-  </joint>
-  <link
-    name="back_left_link">
+    <dynamics friction="0.8" damping="0.5" />
+    <limit lower="-3.14159" upper="3.14159" effort="200" velocity="-1" />
+  </joint>
+  <!--Back Left Wheel-->
+  <link name="back_left_link">
     <inertial>
       <origin
@@ -120,42 +132,35 @@
       <origin
         xyz="0 0 0"
-        rpy="0 0 0" />
+        rpy="${pi} 0 0" />
       <geometry>
         <mesh
           filename="package://yahboom_bot_1/meshes/Ackermann/back_right_link.STL" />
       </geometry>
-      <material
-        name="">
-        <color
-          rgba="0.792156862745098 0.819607843137255 0.933333333333333 1" />
-      </material>
-    </visual>
-    <collision>
-      <origin
-        xyz="0 0 0"
-        rpy="0 0 0" />
-      <geometry>
-        <mesh
-          filename="package://yahboom_bot_1/meshes/Ackermann/back_right_link.STL" />
-      </geometry>
-    </collision>
-  </link>
-  <joint
-    name="back_left_joint"
-    type="continuous">
+      <material name="grey"/>
+    </visual>
+    <collision>
+      <origin
+        xyz="0 0 0"
+        rpy="${pi/2} 0 0" />
+      <geometry>
+        <cylinder radius="0.035" length="0.022" />
+      </geometry>
+    </collision>
+  </link>
+  <joint name="back_left_joint" type="continuous">
     <origin
       xyz="-0.11607 0.08425 0.0125"
       rpy="0 0 0" />
     <parent
-      link="base_link" />
+      link="chassis" />
     <child
       link="back_left_link" />
     <axis
       xyz="0 1 0" />
-    <dynamics
-      damping="0.05" />
-  </joint>
-  <link
-    name="front_left_steer">
+    <dynamics friction="0.8" damping="0.5" />
+    <limit lower="-3.14159" upper="3.14159" effort="200" velocity="-1" />
+  </joint>
+  <!--Front Left Steering Joint-->
+  <link name="front_left_steer">
     <inertial>
       <origin
@@ -181,8 +186,5 @@
       </geometry>
       <material
-        name="">
-        <color
-          rgba="0.082353 0.56078 0 1" />
-      </material>
+        name="grey" />
     </visual>
     <collision>
@@ -196,12 +198,10 @@
     </collision>
   </link>
-  <joint
-    name="front_left_steer_joint"
-    type="revolute">
+  <joint name="front_left_steer_joint" type="revolute">
     <origin
       xyz="0.11922 0.065 0.0262"
       rpy="0 0 0" />
     <parent
-      link="base_link" />
+      link="chassis" />
     <child
       link="front_left_steer" />
@@ -213,9 +213,7 @@
       effort="10"
       velocity="1" />
-    <dynamics
-      damping="0.05" />
-  </joint>
-  <link
-    name="front_left_wheel">
+  </joint>
+  <!--Front Left Wheel Joint-->
+  <link name="front_left_wheel">
     <inertial>
       <origin
@@ -235,28 +233,21 @@
       <origin
         xyz="0 0 0"
-        rpy="0 0 0" />
+        rpy="${pi} 0 0" />
       <geometry>
         <mesh
           filename="package://yahboom_bot_1/meshes/Ackermann/back_right_link.STL" />
       </geometry>
-      <material
-        name="">
-        <color
-          rgba="0.79216 0.81961 0.93333 1" />
-      </material>
-    </visual>
-    <collision>
-      <origin
-        xyz="0 0 0"
-        rpy="0 0 0" />
-      <geometry>
-        <mesh
-          filename="package://yahboom_bot_1/meshes/Ackermann/back_right_link.STL" />
-      </geometry>
-    </collision>
-  </link>
-  <joint
-    name="front_left_wheel_joint"
-    type="continuous">
+      <material name="grey"/>
+    </visual>
+    <collision>
+      <origin
+        xyz="0 0 0"
+        rpy="${pi/2} 0 0" />
+      <geometry>
+        <cylinder radius="0.035" length="0.022" />
+      </geometry>
+    </collision>
+  </link>
+  <joint name="front_left_wheel_joint" type="continuous">
     <origin
       xyz="0.00022897 0.0228 -0.0141"
@@ -267,10 +258,10 @@
       link="front_left_wheel" />
     <axis
-      xyz="0 -1 0" />
-    <dynamics
-      damping="0.05" />
-  </joint>
-  <link
-    name="front_right_steer">
+      xyz="0 1 0" />
+    <dynamics friction="0.8" damping="0.5" />
+    <limit lower="-3.14159" upper="3.14159" effort="200" velocity="-1" />
+  </joint>
+  <!--Front Right Steering Joint-->
+  <link name="front_right_steer">
     <inertial>
       <origin
@@ -290,33 +281,26 @@
       <origin
         xyz="0 0 0"
-        rpy="0 0 0" />
+        rpy="0 0 ${pi}" />
       <geometry>
         <mesh
           filename="package://yahboom_bot_1/meshes/Ackermann/front_left_steer.STL" />
       </geometry>
-      <material
-        name="">
-        <color
-          rgba="0.082353 0.56078 0 1" />
-      </material>
-    </visual>
-    <collision>
-      <origin
-        xyz="0 0 0"
-        rpy="0 0 0" />
-      <geometry>
-        <mesh
-          filename="package://yahboom_bot_1/meshes/Ackermann/front_left_steer.STL" />
-      </geometry>
-    </collision>
-  </link>
-  <joint
-    name="front_right_steer_joint"
-    type="revolute">
+      <material name="grey"/>
+    </visual>
+    <collision>
+      <origin
+        xyz="0 0 0"
+        rpy="0 0 0" />
+      <geometry>
+        <box size="0.015 0.015 0.015" />
+      </geometry>
+    </collision>
+  </link>
+  <joint name="front_right_steer_joint" type="revolute">
     <origin
       xyz="0.11922 -0.065 0.0242"
       rpy="0 0 0" />
     <parent
-      link="base_link" />
+      link="chassis" />
     <child
       link="front_right_steer" />
@@ -328,9 +312,7 @@
       effort="10"
       velocity="1" />
-    <dynamics
-      damping="0.05" />
-  </joint>
-  <link
-    name="front_right_wheel">
+  </joint>
+  <!--Front Right Wheel Joint-->
+  <link name="front_right_wheel">
     <inertial>
       <origin
@@ -355,23 +337,16 @@
           filename="package://yahboom_bot_1/meshes/Ackermann/back_right_link.STL" />
       </geometry>
-      <material
-        name="">
-        <color
-          rgba="0.79216 0.81961 0.93333 1" />
-      </material>
-    </visual>
-    <collision>
-      <origin
-        xyz="0 0 0"
-        rpy="0 0 0" />
-      <geometry>
-        <mesh
-          filename="package://yahboom_bot_1/meshes/Ackermann/back_right_link.STL" />
-      </geometry>
-    </collision>
-  </link>
-  <joint
-    name="front_right_wheel_joint"
-    type="continuous">
+      <material name="grey"/>
+    </visual>
+    <collision>
+      <origin
+        xyz="0 0 0"
+        rpy="${pi/2} 0 0" />
+      <geometry>
+        <cylinder radius="0.035" length="0.022" />
+      </geometry>
+    </collision>
+  </link>
+  <joint name="front_right_wheel_joint" type="continuous">
     <origin
       xyz="-0.00025662 -0.019549 -0.0121"
@@ -383,139 +358,6 @@
     <axis
       xyz="0 1 0" />
-    <dynamics
-      damping="0.05" />
-  </joint>
-  <link
-    name="camera_link">
-    <inertial>
-      <origin
-        xyz="-0.0022507 -5.8908E-06 -0.021168"
-        rpy="0 0 0" />
-      <mass
-        value="0.22414" />
-      <inertia
-        ixx="0.00039172"
-        ixy="2.2482E-08"
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
Commit message: began adding lidar

File: description/gazebo_control.xacro (robot description, xacro)
@@ -89,5 +89,5 @@
             <max_steering_angle>1.570796</max_steering_angle>
             <!-- Max absolute linear speed in m/s -->
-            <max_speed>5</max_speed>
+            <max_speed>20</max_speed>
             <!-- PID tuning -->
             <left_steering_pid_gain>1500 0 1</left_steering_pid_gain>

File: description/robot.urdf.xacro (robot description, xacro)
@@ -5,3 +5,4 @@
   <xacro:include filename="robot_core.xacro" />
   <xacro:include filename="gazebo_control.xacro" />
+  <xacro:include filename="lidar.xacro" />
 </robot>

File: description/robot_core.xacro (robot description, xacro)
@@ -47,5 +47,5 @@
         <parent link="base_link" />
         <child link="chassis_link" />
-        <origin xyz="0.2078 0.0 0.1555" rpy="0 0 0" />
+        <origin xyz="0.0 0.0 0.0" rpy="0 0 0" />
     </joint>
     <!-- FRONT LEFT WHEEL -->
