Commit message: troubleshooting camera and lidar functinality

File: description/OLD_lidar.xacro (robot description, xacro)
@@ -2,16 +2,10 @@
 <robot xmlns:xacro="http://www.ros.org/wiki/xacro">
     <link name="laser_link">
-        <visual>
-            <geometry>
-                <cylinder radius="0.02" length="0.02"/>
-            </geometry>
-        </visual>
-        <collision>
-            <geometry>
-                <cylinder radius="0.02" length="0.02"/>
-            </geometry>
-        </collision>
         <inertial>
-            <mass value="0.01"/>
+            <origin
+                xyz="0 0 0"
+                rpy="0 0 0" />
+            <mass
+                value="0.01" />
             <inertia
                 ixx="0"
@@ -22,4 +16,27 @@
                 izz="0" />
         </inertial>
+        <visual>
+            <origin
+                xyz="0 0 0"
+                rpy="0 0 0" />
+            <geometry>
+                <mesh
+                filename="package://yahboom_bot_1/meshes/Ackermann/laser_link.STL" />
+            </geometry>
+            <material
+                name="">
+                <color
+                rgba="1 1 1 1" />
+            </material>
+        </visual>
+        <collision>
+            <origin
+                xyz="0 0 0"
+                rpy="0 0 0" />
+            <geometry>
+                <mesh
+                filename="package://yahboom_bot_1/meshes/Ackermann/laser_link.STL" />
+            </geometry>
+        </collision>
     </link>
     <joint name="laser_joint" type="fixed">
@@ -30,5 +47,4 @@
     </joint>
     <gazebo reference="laser_link">
-        <material>Gazebo/Red</material>
         <sensor name="laser" type="ray">
             <update_rate>10</update_rate>
@@ -44,6 +60,6 @@
                 </scan>
                 <range>
-                    <min>0.021</min>
-                    <max>5.0</max>
+                    <min>0.1</min>
+                    <max>10.0</max>
                 </range>
             </ray>

File: description/gazebo_control.xacro (robot description, xacro)
@@ -91,9 +91,9 @@
             <max_speed>20</max_speed>
             <!-- PID tuning -->
-            <left_steering_pid_gain>1500 0 1</left_steering_pid_gain>
+            <left_steering_pid_gain>150 0 1</left_steering_pid_gain>
             <left_steering_i_range>0 0</left_steering_i_range>
-            <right_steering_pid_gain>1500 0 1</right_steering_pid_gain>
+            <right_steering_pid_gain>150 0 1</right_steering_pid_gain>
             <right_steering_i_range>0 0</right_steering_i_range>
-            <linear_velocity_pid_gain>1500 0 1</linear_velocity_pid_gain>
+            <linear_velocity_pid_gain>150 1 1</linear_velocity_pid_gain>
             <linear_velocity_i_range>0 0</linear_velocity_i_range>
             <!-- output -->

File: description/robot.urdf.xacro (robot description, xacro)
@@ -1,8 +1,7 @@
 <?xml version="1.0" encoding="utf-8"?>
 <robot name="yahboom_bot_1" xmlns:xacro="http://ros.org/wiki/xacro">
-  <!-- <xacro:include filename="TEST_ack_tweak.xacro" />
-  <xacro:include filename="TEST_gazebo_ack.xacro" /> -->
   <xacro:include filename="robot_core.xacro" />
   <xacro:include filename="gazebo_control.xacro" />
   <xacro:include filename="lidar.xacro" />
+  <xacro:include filename="camera.xacro" />
 </robot>
