Commit message: got the camera and lidar both workinggit add .! I dont know why this worked but I pasted the camera xacro from articulated robotics. the lidar was fixed a couple of commits ago by correcting the plugin name

File: description/camera.xacro (robot description, xacro)
@@ -1,64 +1,50 @@
 <?xml version="1.0"?>
-<robot xmlns:xacro="http://www.ros.org/wiki/xacro">
+<robot xmlns:xacro="http://www.ros.org/wiki/xacro" >
+    <joint name="camera_joint" type="fixed">
+        <parent link="chassis_link"/>
+        <child link="camera_link"/>
+        <origin xyz="0.276 0 0.181" rpy="0 0.18 0"/>
+    </joint>
     <link name="camera_link">
         <visual>
             <geometry>
-                <cylinder radius="0.02" length="0.02"/>
+                <box size="0.010 0.03 0.03"/>
             </geometry>
+            <material name="black"/>
         </visual>
-        <collision>
+        <visual>
+            <origin xyz="0 0 -0.05"/>
             <geometry>
-                <cylinder radius="0.02" length="0.02"/>
+                <cylinder radius="0.002" length="0.1"/>
             </geometry>
-        </collision>
-        <inertial>
-            <mass value="0.01"/>
-            <inertia
-                ixx="0"
-                ixy="0"
-                ixz="0"
-                iyy="0"
-                iyz="0"
-                izz="0" />
-        </inertial>
+            <material name="black"/>
+        </visual>
     </link>
-    <joint name="camera_joint" type="fixed">
-        <origin xyz="0.1 0 0.075" rpy="0 ${pi/2} 0" />
-        <parent link="base_link" />
-        <child link="camera_link" />
-        <axis xyz="0 0 0" />
+    <joint name="camera_optical_joint" type="fixed">
+        <parent link="camera_link"/>
+        <child link="camera_link_optical"/>
+        <origin xyz="0 0 0" rpy="${-pi/2} 0 ${-pi/2}"/>
     </joint>
     <link name="camera_link_optical"></link>
-    <joint name="camera_optical_joint" type="fixed">
-        <origin xyz="0 0 0" rpy="${pi} ${pi} ${pi/2}" />
-        <parent link="camera_link" />
-        <child link="camera_link_optical" />
-    </joint>
     <gazebo reference="camera_link">
-        <material>Gazebo/Red</material>
-        <sensor type="camera" name="my_camera">
+        <material>Gazebo/Black</material>
+        <sensor name="camera" type="camera">
+            <pose> 0 0 0 0 0 0 </pose>
+            <visualize>true</visualize>
             <update_rate>10</update_rate>
-            <visualize>true</visualize>
-            <camera name="cam">
-                <horizontal_fov>1.3962634</horizontal_fov>
+            <camera>
+                <horizontal_fov>1.089</horizontal_fov>
                 <image>
+                    <format>R8G8B8</format>
                     <width>640</width>
                     <height>480</height>
-                    <format>R8G8B8</format>
                 </image>
                 <clip>
-                    <near>0.1</near>
-                    <far>100.0</far>
+                    <near>0.05</near>
+                    <far>8.0</far>
                 </clip>
-                <noise>
-                    <type>gaussian</type>
-                    <mean>0.0</mean>
-                    <stddev>0.01</stddev>
-                </noise>
             </camera>
             <plugin name="camera_controller" filename="libgazebo_ros_camera.so">
                 <frame_name>camera_link_optical</frame_name>
-                <min_depth>0.1</min_depth>
-                <max_depth>100.0</max_depth>
             </plugin>
         </sensor>

Commit message: added depth camera functionality, continued troubleshooting inertia/PID issues of yahboom xacro with real inertia values in robot_core_TEST

File: description/camera.xacro (robot description, xacro)
@@ -28,6 +28,6 @@
     <link name="camera_link_optical"></link>
     <gazebo reference="camera_link">
-        <material>Gazebo/Black</material>
-        <sensor name="camera" type="camera">
+        <material>Gazebo/Red</material>
+        <sensor name="camera" type="depth">
             <pose> 0 0 0 0 0 0 </pose>
             <visualize>true</visualize>
@@ -36,5 +36,5 @@
                 <horizontal_fov>1.089</horizontal_fov>
                 <image>
-                    <format>R8G8B8</format>
+                    <format>B8G8R8</format>
                     <width>640</width>
                     <height>480</height>
@@ -47,4 +47,6 @@
             <plugin name="camera_controller" filename="libgazebo_ros_camera.so">
                 <frame_name>camera_link_optical</frame_name>
+                <min_depth>0.1</min_depth>
+                <max_depth>100.0</max_depth>
             </plugin>
         </sensor>

File: description/robot.urdf.xacro (robot description, xacro)
@@ -1,6 +1,7 @@
 <?xml version="1.0" encoding="utf-8"?>
 <robot name="yahboom_bot_1" xmlns:xacro="http://ros.org/wiki/xacro">
-  <xacro:include filename="robot_core_TEST.xacro" />
-  <xacro:include filename="gazebo_control.xacro" />
+  <xacro:include filename="robot_core.xacro" />
+  <!-- <xacro:include filename="gazebo_control.xacro" /> -->
+  <xacro:include filename="ros2_control.xacro" />
   <xacro:include filename="lidar.xacro" />
   <xacro:include filename="camera.xacro" />

File: description/robot_core_TEST.xacro (robot description, xacro)
@@ -1,11 +1,11 @@
 <?xml version="1.0"?>
 <robot xmlns:xacro="http://www.ros.org/wiki/xacro">
-    <xacro:property name="body_mass" value="25.0" />
-    <xacro:property name="body_width" value="0.3" />
-    <xacro:property name="body_length" value="0.10" />
-    <xacro:property name="body_depth" value="0.75" />
-    <xacro:property name="wheel_radius" value="0.14" />
-    <xacro:property name="wheel_thickness" value="0.14" />
-    <xacro:property name="wheel_mass" value="3.0" />
+    <xacro:property name="body_mass" value="0.52" />
+    <xacro:property name="body_width" value="0.075" />
+    <xacro:property name="body_length" value="0.15" />
+    <xacro:property name="body_depth" value="0.05" />
+    <xacro:property name="wheel_radius" value="0.022" />
+    <xacro:property name="wheel_thickness" value="0.022" />
+    <xacro:property name="wheel_mass" value="0.5" />
     <xacro:property name="steering_mass" value="0.01" />
     <!-- BASE -->
@@ -23,5 +23,5 @@
         <inertial>
             <origin xyz="0 0 0" rpy="0 0 0" />
-            <mass value="24.73" />
+            <mass value="${body_mass}" />
             <inertia ixx="${body_mass/12 * (body_width*body_width + body_length*body_length)}"
                 ixy="0" ixz="0"
@@ -79,5 +79,5 @@
     <link name="fr_left_wheel_link">
         <inertial>
-            <origin xyz="-6.1417E-08 -0.0048115 4.113E-08" rpy="0 0 0" />
+            <origin xyz="0 0 0" rpy="0 0 0" />
             <mass value="${wheel_mass}" />
             <inertia
@@ -142,5 +142,5 @@
     <link name="fr_right_wheel_link">
         <inertial>
-            <origin xyz="5.5753E-08 0.0015615 -5.0453E-08" rpy="0 0 0" />
+            <origin xyz="0 0 0" rpy="0 0 0" />
             <mass value="${wheel_mass}" />
             <inertia
@@ -177,5 +177,5 @@
     <link name="re_left_wheel_link">
         <inertial>
-            <origin xyz="-6.87042718550135E-08 -0.00156153690070754 3.00324059371304E-08" rpy="0 0 0" />
+            <origin xyz="0 0 0" rpy="0 0 0" />
             <mass value="${wheel_mass}" />
             <inertia
@@ -216,5 +216,5 @@
         <inertial>
             <origin
-                xyz="3.8959E-08 0.0015615 -6.3774E-08"
+                xyz="0 0 0"
                 rpy="0 0 0" />
             <mass value="${wheel_mass}" />
