Commit message: ackermann steering now working with ros2_controlgit add .

File: description/ack_ros2_control.xacro (robot description, xacro)
@@ -21,8 +21,24 @@
             <state_interface name="velocity"/>
         </joint>
+        <joint name="fr_left_steer_joint">
+            <command_interface name="position">
+                <param name="min">-1.0</param>
+                <param name="max">1.0</param>
+            </command_interface>
+            <state_interface name="position"/>
+            <state_interface name="velocity"/>
+        </joint>
+        <joint name="fr_right_steer_joint">
+            <command_interface name="position">
+                <param name="min">-1.0</param>
+                <param name="max">1.0</param>
+            </command_interface>
+            <state_interface name="position"/>
+            <state_interface name="velocity"/>
+        </joint>
     </ros2_control>
     <gazebo>
         <plugin filename="libgazebo_ros2_control.so" name="gazebo_ros2_control">
-            <parameters>$(find yahboom_bot_1)/config/controllers.yaml</parameters>
+            <parameters>$(find yahboom_bot_1)/config/ack_controllers.yaml</parameters>
         </plugin>
     </gazebo>

File: description/robot.urdf.xacro (robot description, xacro)
@@ -2,6 +2,6 @@
 <robot name="yahboom_bot_1" xmlns:xacro="http://ros.org/wiki/xacro">
   <xacro:include filename="robot_core.xacro" />
-  <xacro:include filename="gazebo_control.xacro" />
-  <!-- <xacro:include filename="ros2_control.xacro" /> -->
+  <!-- <xacro:include filename="gazebo_control.xacro" /> -->
+  <xacro:include filename="ack_ros2_control.xacro" />
   <xacro:include filename="lidar.xacro" />
   <xacro:include filename="camera.xacro" />
